Commit message: update xacro

File: logiee-s-tc_sensor_kit_description/urdf/sensor_kit.xacro (robot description, xacro)
@@ -20,45 +20,34 @@
     <xacro:property name="calibration" value="${xacro.load_yaml('$(arg config_dir)/sensor_kit_calibration.yaml')}"/>
     <!-- lidar -->
-    <xacro:VLS-128 parent="sensor_kit_base_link" name="velodyne_top" topic="/points_raw" hz="10" samples="220" gpu="$(arg gpu)">
+    <xacro:VLP-16 parent="sensor_kit_base_link" name="/velodyne_front" topic="/sensing/lidar/front/pointcloud_ex" hz="10" samples="220" gpu="$(arg gpu)">
       <origin
-        xyz="${calibration['sensor_kit_base_link']['velodyne_top_base_link']['x']}
-             ${calibration['sensor_kit_base_link']['velodyne_top_base_link']['y']}
-             ${calibration['sensor_kit_base_link']['velodyne_top_base_link']['z']}"
-        rpy="${calibration['sensor_kit_base_link']['velodyne_top_base_link']['roll']}
-             ${calibration['sensor_kit_base_link']['velodyne_top_base_link']['pitch']}
-             ${calibration['sensor_kit_base_link']['velodyne_top_base_link']['yaw']}"
+        xyz="${calibration['sensor_kit_base_link']['velodyne_front_base_link']['x']}
+             ${calibration['sensor_kit_base_link']['velodyne_front_base_link']['y']}
+             ${calibration['sensor_kit_base_link']['velodyne_front_base_link']['z']}"
+        rpy="${calibration['sensor_kit_base_link']['velodyne_front_base_link']['roll']}
+             ${calibration['sensor_kit_base_link']['velodyne_front_base_link']['pitch']}
+             ${calibration['sensor_kit_base_link']['velodyne_front_base_link']['yaw']}"
       />
     </xacro:VLS-128>
-    <xacro:VLP-16 parent="sensor_kit_base_link" name="velodyne_left" topic="/points_raw" hz="10" samples="220" gpu="$(arg gpu)">
+    <xacro:VLP-16 parent="sensor_kit_base_link" name="velodyne_rear" topic="/sensing/lidar/rear/pointcloud_ex" hz="10" samples="220" gpu="$(arg gpu)">
       <origin
-        xyz="${calibration['sensor_kit_base_link']['velodyne_left_base_link']['x']}
-             ${calibration['sensor_kit_base_link']['velodyne_left_base_link']['y']}
-             ${calibration['sensor_kit_base_link']['velodyne_left_base_link']['z']}"
-        rpy="${calibration['sensor_kit_base_link']['velodyne_left_base_link']['roll']}
-             ${calibration['sensor_kit_base_link']['velodyne_left_base_link']['pitch']}
-             ${calibration['sensor_kit_base_link']['velodyne_left_base_link']['yaw']}"
+        xyz="${calibration['sensor_kit_base_link']['velodyne_rear_base_link']['x']}
+             ${calibration['sensor_kit_base_link']['velodyne_rear_base_link']['y']}
+             ${calibration['sensor_kit_base_link']['velodyne_rear_base_link']['z']}"
+        rpy="${calibration['sensor_kit_base_link']['velodyne_rear_base_link']['roll']}
+             ${calibration['sensor_kit_base_link']['velodyne_rear_base_link']['pitch']}
+             ${calibration['sensor_kit_base_link']['velodyne_rear_base_link']['yaw']}"
       />
-    </xacro:VLP-16>
-    <xacro:VLP-16 parent="sensor_kit_base_link" name="velodyne_right" topic="/points_raw" hz="10" samples="220" gpu="$(arg gpu)">
-      <origin
-        xyz="${calibration['sensor_kit_base_link']['velodyne_right_base_link']['x']}
-             ${calibration['sensor_kit_base_link']['velodyne_right_base_link']['y']}
-             ${calibration['sensor_kit_base_link']['velodyne_right_base_link']['z']}"
-        rpy="${calibration['sensor_kit_base_link']['velodyne_right_base_link']['roll']}
-             ${calibration['sensor_kit_base_link']['velodyne_right_base_link']['pitch']}
-             ${calibration['sensor_kit_base_link']['velodyne_right_base_link']['yaw']}"
-      />
-    </xacro:VLP-16>
     <!-- camera -->
     <xacro:monocular_camera_macro
-      name="traffic_light_right_camera/camera"
+      name="front_cam_base_link"
       parent="sensor_kit_base_link"
       namespace=""
-      x="${calibration['sensor_kit_base_link']['traffic_light_right_camera/camera_link']['x']}"
-      y="${calibration['sensor_kit_base_link']['traffic_light_right_camera/camera_link']['y']}"
-      z="${calibration['sensor_kit_base_link']['traffic_light_right_camera/camera_link']['z']}"
-      roll="${calibration['sensor_kit_base_link']['traffic_light_right_camera/camera_link']['roll']}"
-      pitch="${calibration['sensor_kit_base_link']['traffic_light_right_camera/camera_link']['pitch']}"
-      yaw="${calibration['sensor_kit_base_link']['traffic_light_right_camera/camera_link']['yaw']}"
+      x="${calibration['sensor_kit_base_link']['front_cam_base_link2']['x']}"
+      y="${calibration['sensor_kit_base_link']['front_cam_base_link2']['y']}"
+      z="${calibration['sensor_kit_base_link']['front_cam_base_link2']['z']}"
+      roll="${calibration['sensor_kit_base_link']['front_cam_base_link2']['roll']}"
+      pitch="${calibration['sensor_kit_base_link']['front_cam_base_link2']['pitch']}"
+      yaw="${calibration['sensor_kit_base_link']['front_cam_base_link2']['yaw']}"
       fps="30"
       width="800"
@@ -67,103 +56,13 @@
     />
     <xacro:monocular_camera_macro
-      name="traffic_light_left_camera/camera"
+      name="front_c1_cam_base_link2"
       parent="sensor_kit_base_link"
       namespace=""
-      x="${calibration['sensor_kit_base_link']['traffic_light_left_camera/camera_link']['x']}"
-      y="${calibration['sensor_kit_base_link']['traffic_light_left_camera/camera_link']['y']}"
-      z="${calibration['sensor_kit_base_link']['traffic_light_left_camera/camera_link']['z']}"
-      roll="${calibration['sensor_kit_base_link']['traffic_light_left_camera/camera_link']['roll']}"
-      pitch="${calibration['sensor_kit_base_link']['traffic_light_left_camera/camera_link']['pitch']}"
-      yaw="${calibration['sensor_kit_base_link']['traffic_light_left_camera/camera_link']['yaw']}"
-      fps="30"
-      width="800"
-      height="400"
-      fov="1.3"
-    />
-    <xacro:monocular_camera_macro
-      name="camera0/camera"
-      parent="sensor_kit_base_link"
-      namespace=""
-      x="${calibration['sensor_kit_base_link']['camera0/camera_link']['x']}"
-      y="${calibration['sensor_kit_base_link']['camera0/camera_link']['y']}"
-      z="${calibration['sensor_kit_base_link']['camera0/camera_link']['z']}"
-      roll="${calibration['sensor_kit_base_link']['camera0/camera_link']['roll']}"
-      pitch="${calibration['sensor_kit_base_link']['camera0/camera_link']['pitch']}"
-      yaw="${calibration['sensor_kit_base_link']['camera0/camera_link']['yaw']}"
-      fps="30"
-      width="800"
-      height="400"
-      fov="1.3"
-    />
-    <xacro:monocular_camera_macro
-      name="camera1/camera"
-      parent="sensor_kit_base_link"
-      namespace=""
-      x="${calibration['sensor_kit_base_link']['camera1/camera_link']['x']}"
-      y="${calibration['sensor_kit_base_link']['camera1/camera_link']['y']}"
-      z="${calibration['sensor_kit_base_link']['camera1/camera_link']['z']}"
-      roll="${calibration['sensor_kit_base_link']['camera1/camera_link']['roll']}"
-      pitch="${calibration['sensor_kit_base_link']['camera1/camera_link']['pitch']}"
-      yaw="${calibration['sensor_kit_base_link']['camera1/camera_link']['yaw']}"
-      fps="30"
-      width="800"
-      height="400"
-      fov="1.3"
-    />
-    <xacro:monocular_camera_macro
-      name="camera2/camera"
-      parent="sensor_kit_base_link"
-      namespace=""
-      x="${calibration['sensor_kit_base_link']['camera2/camera_link']['x']}"
-      y="${calibration['sensor_kit_base_link']['camera2/camera_link']['y']}"
-      z="${calibration['sensor_kit_base_link']['camera2/camera_link']['z']}"
-      roll="${calibration['sensor_kit_base_link']['camera2/camera_link']['roll']}"
-      pitch="${calibration['sensor_kit_base_link']['camera2/camera_link']['pitch']}"
-      yaw="${calibration['sensor_kit_base_link']['camera2/camera_link']['yaw']}"
-      fps="30"
-      width="800"
-      height="400"
-      fov="1.3"
-    />
-    <xacro:monocular_camera_macro
-      name="camera3/camera"
-      parent="sensor_kit_base_link"
-      namespace=""
-      x="${calibration['sensor_kit_base_link']['camera3/camera_link']['x']}"
-      y="${calibration['sensor_kit_base_link']['camera3/camera_link']['y']}"
-      z="${calibration['sensor_kit_base_link']['camera3/camera_link']['z']}"
-      roll="${calibration['sensor_kit_base_link']['camera3/camera_link']['roll']}"
-      pitch="${calibration['sensor_kit_base_link']['camera3/camera_link']['pitch']}"
-      yaw="${calibration['sensor_kit_base_link']['camera3/camera_link']['yaw']}"
-      fps="30"
-      width="800"
-      height="400"
-      fov="1.3"
-    />
-    <xacro:monocular_camera_macro
-      name="camera4/camera"
-      parent="sensor_kit_base_link"
-      namespace=""
-      x="${calibration['sensor_kit_base_link']['camera4/camera_link']['x']}"
-      y="${calibration['sensor_kit_base_link']['camera4/camera_link']['y']}"
-      z="${calibration['sensor_kit_base_link']['camera4/camera_link']['z']}"
-      roll="${calibration['sensor_kit_base_link']['camera4/camera_link']['roll']}"
-      pitch="${calibration['sensor_kit_base_link']['camera4/camera_link']['pitch']}"
-      yaw="${calibration['sensor_kit_base_link']['camera4/camera_link']['yaw']}"
-      fps="30"
-      width="800"
-      height="400"
-      fov="1.3"
-    />
-    <xacro:monocular_camera_macro
-      name="camera5/camera"
-      parent="sensor_kit_base_link"
-      namespace=""
-      x="${calibration['sensor_kit_base_link']['camera5/camera_link']['x']}"
-      y="${calibration['sensor_kit_base_link']['camera5/camera_link']['y']}"
-      z="${calibration['sensor_kit_base_link']['camera5/camera_link']['z']}"
-      roll="${calibration['sensor_kit_base_link']['camera5/camera_link']['roll']}"
-      pitch="${calibration['sensor_kit_base_link']['camera5/camera_link']['pitch']}"
-      yaw="${calibration['sensor_kit_base_link']['camera5/camera_link']['yaw']}"
+      x="${calibration['sensor_kit_base_link']['front_c1_cam_base_link2']['x']}"
+      y="${calibration['sensor_kit_base_link']['front_c1_cam_base_link2']['y']}"
+      z="${calibration['sensor_kit_base_link']['front_c1_cam_base_link2']['z']}"
+      roll="${calibration['sensor_kit_base_link']['front_c1_cam_base_link2']['roll']}"
+      pitch="${calibration['sensor_kit_base_link']['front_c1_cam_base_link2']['pitch']}"
+      yaw="${calibration['sensor_kit_base_link']['front_c1_cam_base_link2']['yaw']}"
       fps="30"
       width="800"
@@ -172,5 +71,5 @@
     />
     <!-- gnss -->
-    <xacro:imu_macro
+    <!-- <xacro:imu_macro
       name="gnss"
       parent="sensor_kit_base_link"
@@ -183,16 +82,16 @@
       yaw="${calibration['sensor_kit_base_link']['gnss_link']['yaw']}"
       fps="100"
-    />
+    /> -->
     <!-- imu -->
     <xacro:imu_macro
-      name="tamagawa/imu"
+      name="imu_link"
       parent="sensor_kit_base_link"
       namespace=""
-      x="${calibration['sensor_kit_base_link']['tamagawa/imu_link']['x']}"
-      y="${calibration['sensor_kit_base_link']['tamagawa/imu_link']['y']}"
-      z="${calibration['sensor_kit_base_link']['tamagawa/imu_link']['z']}"
-      roll="${calibration['sensor_kit_base_link']['tamagawa/imu_link']['roll']}"
-      pitch="${calibration['sensor_kit_base_link']['tamagawa/imu_link']['pitch']}"
-      yaw="${calibration['sensor_kit_base_link']['tamagawa/imu_link']['yaw']}"
+      x="${calibration['sensor_kit_base_link']['imu_link2']['x']}"
+      y="${calibration['sensor_kit_base_link']['imu_link2']['y']}"
+      z="${calibration['sensor_kit_base_link']['imu_link2']['z']}"
+      roll="${calibration['sensor_kit_base_link']['imu_link2']['roll']}"
+      pitch="${calibration['sensor_kit_base_link']['imu_link2']['pitch']}"
+      yaw="${calibration['sensor_kit_base_link']['imu_link2']['yaw']}"
       fps="100"
     />

File: logiee-s-tc_sensor_kit_description/urdf/sensors.xacro (robot description, xacro)
@@ -6,4 +6,14 @@
   <xacro:include filename="$(find imu_description)/urdf/imu.xacro"/>
   <xacro:property name="calibration" value="${load_yaml('$(arg config_dir)/sensors_calibration.yaml')}"/>
+  <!-- <xacro:include filename="sensor_kit.xacro"/>
+  <xacro:sensor_kit_macro
+    parent="base_link"
+    x="${calibration['base_link']['sensor_kit_base_link']['x']}"
+    y="${calibration['base_link']['sensor_kit_base_link']['y']}"
+    z="${calibration['base_link']['sensor_kit_base_link']['z']}"
+    roll="${calibration['base_link']['sensor_kit_base_link']['roll']}"
+    pitch="${calibration['base_link']['sensor_kit_base_link']['pitch']}"
+    yaw="${calibration['base_link']['sensor_kit_base_link']['yaw']}"
+  /> -->
   <!-- lidar -->
   <xacro:VLP-16 parent="base_link" name="velodyne_rear" topic="/sensing/lidar/rear/pointcloud_ex" hz="10" samples="220" gpu="$(arg gpu)">

Commit message: use sensor_kit_base_link

File: logiee-s-tc_sensor_kit_description/urdf/sensor_kit.xacro (robot description, xacro)
@@ -20,34 +20,35 @@
     <xacro:property name="calibration" value="${xacro.load_yaml('$(arg config_dir)/sensor_kit_calibration.yaml')}"/>
     <!-- lidar -->
-    <xacro:VLP-16 parent="sensor_kit_base_link" name="/velodyne_front" topic="/sensing/lidar/front/pointcloud_ex" hz="10" samples="220" gpu="$(arg gpu)">
+    <xacro:VLP-16 parent="sensor_kit_base_link" name="velodyne_front" topic="/sensing/lidar/front/pointcloud_ex" hz="10" samples="220" gpu="$(arg gpu)">
       <origin
-        xyz="${calibration['sensor_kit_base_link']['velodyne_front_base_link']['x']}
-             ${calibration['sensor_kit_base_link']['velodyne_front_base_link']['y']}
-             ${calibration['sensor_kit_base_link']['velodyne_front_base_link']['z']}"
-        rpy="${calibration['sensor_kit_base_link']['velodyne_front_base_link']['roll']}
-             ${calibration['sensor_kit_base_link']['velodyne_front_base_link']['pitch']}
-             ${calibration['sensor_kit_base_link']['velodyne_front_base_link']['yaw']}"
+        xyz="${calibration['sensor_kit_base_link2velodyne_front']['x']}
+             ${calibration['sensor_kit_base_link2velodyne_front']['y']}
+             ${calibration['sensor_kit_base_link2velodyne_front']['z']}"
+        rpy="${calibration['sensor_kit_base_link2velodyne_front']['roll']}
+             ${calibration['sensor_kit_base_link2velodyne_front']['pitch']}
+             ${calibration['sensor_kit_base_link2velodyne_front']['yaw']}"
       />
-    </xacro:VLS-128>
+    </xacro:VLP-16>
     <xacro:VLP-16 parent="sensor_kit_base_link" name="velodyne_rear" topic="/sensing/lidar/rear/pointcloud_ex" hz="10" samples="220" gpu="$(arg gpu)">
       <origin
-        xyz="${calibration['sensor_kit_base_link']['velodyne_rear_base_link']['x']}
-             ${calibration['sensor_kit_base_link']['velodyne_rear_base_link']['y']}
-             ${calibration['sensor_kit_base_link']['velodyne_rear_base_link']['z']}"
-        rpy="${calibration['sensor_kit_base_link']['velodyne_rear_base_link']['roll']}
-             ${calibration['sensor_kit_base_link']['velodyne_rear_base_link']['pitch']}
-             ${calibration['sensor_kit_base_link']['velodyne_rear_base_link']['yaw']}"
+        xyz="${calibration['sensor_kit_base_link2velodyne_rear']['x']}
+             ${calibration['sensor_kit_base_link2velodyne_rear']['y']}
+             ${calibration['sensor_kit_base_link2velodyne_rear']['z']}"
+        rpy="${calibration['sensor_kit_base_link2velodyne_rear']['roll']}
+             ${calibration['sensor_kit_base_link2velodyne_rear']['pitch']}
+             ${calibration['sensor_kit_base_link2velodyne_rear']['yaw']}"
       />
+    </xacro:VLP-16>
     <!-- camera -->
     <xacro:monocular_camera_macro
-      name="front_cam_base_link"
+      name="front_cam_base"
       parent="sensor_kit_base_link"
       namespace=""
-      x="${calibration['sensor_kit_base_link']['front_cam_base_link2']['x']}"
-      y="${calibration['sensor_kit_base_link']['front_cam_base_link2']['y']}"
-      z="${calibration['sensor_kit_base_link']['front_cam_base_link2']['z']}"
-      roll="${calibration['sensor_kit_base_link']['front_cam_base_link2']['roll']}"
-      pitch="${calibration['sensor_kit_base_link']['front_cam_base_link2']['pitch']}"
-      yaw="${calibration['sensor_kit_base_link']['front_cam_base_link2']['yaw']}"
+      x="${calibration['sensor_kit_base_link2front_default_cam']['x']}"
+      y="${calibration['sensor_kit_base_link2front_default_cam']['y']}"
+      z="${calibration['sensor_kit_base_link2front_default_cam']['z']}"
+      roll="${calibration['sensor_kit_base_link2front_default_cam']['roll']}"
+      pitch="${calibration['sensor_kit_base_link2front_default_cam']['pitch']}"
+      yaw="${calibration['sensor_kit_base_link2front_default_cam']['yaw']}"
       fps="30"
       width="800"
@@ -56,13 +57,13 @@
     />
     <xacro:monocular_camera_macro
-      name="front_c1_cam_base_link2"
+      name="front_c1_cam"
       parent="sensor_kit_base_link"
       namespace=""
-      x="${calibration['sensor_kit_base_link']['front_c1_cam_base_link2']['x']}"
-      y="${calibration['sensor_kit_base_link']['front_c1_cam_base_link2']['y']}"
-      z="${calibration['sensor_kit_base_link']['front_c1_cam_base_link2']['z']}"
-      roll="${calibration['sensor_kit_base_link']['front_c1_cam_base_link2']['roll']}"
-      pitch="${calibration['sensor_kit_base_link']['front_c1_cam_base_link2']['pitch']}"
-      yaw="${calibration['sensor_kit_base_link']['front_c1_cam_base_link2']['yaw']}"
+      x="${calibration['sensor_kit_base_link2front_c1_cam']['x']}"
+      y="${calibration['sensor_kit_base_link2front_c1_cam']['y']}"
+      z="${calibration['sensor_kit_base_link2front_c1_cam']['z']}"
+      roll="${calibration['sensor_kit_base_link2front_c1_cam']['roll']}"
+      pitch="${calibration['sensor_kit_base_link2front_c1_cam']['pitch']}"
+      yaw="${calibration['sensor_kit_base_link2front_c1_cam']['yaw']}"
       fps="30"
       width="800"
@@ -88,10 +89,10 @@
       parent="sensor_kit_base_link"
       namespace=""
-      x="${calibration['sensor_kit_base_link']['imu_link2']['x']}"
-      y="${calibration['sensor_kit_base_link']['imu_link2']['y']}"
-      z="${calibration['sensor_kit_base_link']['imu_link2']['z']}"
-      roll="${calibration['sensor_kit_base_link']['imu_link2']['roll']}"
-      pitch="${calibration['sensor_kit_base_link']['imu_link2']['pitch']}"
-      yaw="${calibration['sensor_kit_base_link']['imu_link2']['yaw']}"
+      x="${calibration['sensor_kit_base_link2imu']['x']}"
+      y="${calibration['sensor_kit_base_link2imu']['y']}"
+      z="${calibration['sensor_kit_base_link2imu']['z']}"
+      roll="${calibration['sensor_kit_base_link2imu']['roll']}"
+      pitch="${calibration['sensor_kit_base_link2imu']['pitch']}"
+      yaw="${calibration['sensor_kit_base_link2imu']['yaw']}"
       fps="100"
     />

File: logiee-s-tc_sensor_kit_description/urdf/sensors.xacro (robot description, xacro)
@@ -1,42 +1,10 @@
 <?xml version="1.0"?>
-<robot name="vehicle" xmlns:xacro="http://ros.org/wiki/xacro">
+<robot name="vehicle"
+  xmlns:xacro="http://ros.org/wiki/xacro">
   <xacro:arg name="config_dir" default="$(find logiee-s-tc_sensor_kit_description)/config"/>
-  <xacro:arg name="gpu" default="false"/>
-  <xacro:include filename="$(find velodyne_description)/urdf/VLP-16.urdf.xacro"/>
-  <xacro:include filename="$(find imu_description)/urdf/imu.xacro"/>
+  <xacro:include filename="$(find logiee-s-tc_sensor_kit_description)/urdf/sensor_kit.xacro"/>
   <xacro:property name="calibration" value="${load_yaml('$(arg config_dir)/sensors_calibration.yaml')}"/>
-  <!-- <xacro:include filename="sensor_kit.xacro"/>
-  <xacro:sensor_kit_macro
-    parent="base_link"
-    x="${calibration['base_link']['sensor_kit_base_link']['x']}"
-    y="${calibration['base_link']['sensor_kit_base_link']['y']}"
-    z="${calibration['base_link']['sensor_kit_base_link']['z']}"
-    roll="${calibration['base_link']['sensor_kit_base_link']['roll']}"
-    pitch="${calibration['base_link']['sensor_kit_base_link']['pitch']}"
-    yaw="${calibration['base_link']['sensor_kit_base_link']['yaw']}"
-  /> -->
-  <!-- lidar -->
-  <xacro:VLP-16 parent="base_link" name="velodyne_rear" topic="/sensing/lidar/rear/pointcloud_ex" hz="10" samples="220" gpu="$(arg gpu)">
-    <origin
-      xyz="${calibration['base_link']['velodyne_rear_base_link']['x']}
-           ${calibration['base_link']['velodyne_rear_base_link']['y']}
-           ${calibration['base_link']['velodyne_rear_base_link']['z']}"
-      rpy="${calibration['base_link']['velodyne_rear_base_link']['roll']}
-           ${calibration['base_link']['velodyne_rear_base_link']['pitch']}
-           ${calibration['base_link']['velodyne_rear_base_link']['yaw']}"
-    />
-  </xacro:VLP-16>
-  <xacro:VLP-16 parent="base_link" name="velodyne_front" topic="/sensing/lidar/front/pointcloud_ex" hz="10" samples="220" gpu="$(arg gpu)">
-    <origin
-      xyz="${calibration['base_link']['velodyne_front_base_link']['x']}
-           ${calibration['base_link']['velodyne_front_base_link']['y']}
-           ${calibration['base_link']['velodyne_front_base_link']['z']}"
-      rpy="${calibration['base_link']['velodyne_front_base_link']['roll']}
-           ${calibration['base_link']['velodyne_front_base_link']['pitch']}
-           ${calibration['base_link']['velodyne_front_base_link']['yaw']}"
-    />
-  </xacro:VLP-16>
-  <!-- IMU -->
-  <xacro:imu_macro
+  <xacro:sensor_kit_macro parent="base_link" x="${calibration['base_link2sensor_kit_base_link']['x']}" y="${calibration['base_link2sensor_kit_base_link']['y']}" z="${calibration['base_link2sensor_kit_base_link']['z']}" roll="${calibration['base_link2sensor_kit_base_link']['roll']}" pitch="${calibration['base_link2sensor_kit_base_link']['pitch']}" yaw="${calibration['base_link2sensor_kit_base_link']['yaw']}" />
+  <!-- <xacro:imu_macro
     name="imu_bottom"
     parent="base_link"
@@ -49,28 +17,4 @@
     yaw="${calibration['base_link']['imu_bottom_link']['yaw']}"
     fps="100"
-  />
-  <!-- <xacro:imu_macro
-    name="sensor"
-    parent="base_link"
-    namespace=""
-    x="${calibration['base_link']['sensor']['x']}"
-    y="${calibration['base_link']['sensor']['y']}"
-    z="${calibration['base_link']['sensor']['z']}"
-    roll="${calibration['base_link']['sensor']['roll']}"
-    pitch="${calibration['base_link']['sensor']['pitch']}"
-    yaw="${calibration['base_link']['sensor']['yaw']}"
-    fps="100"
-  /> -->
-  <!-- <xacro
-    name="sensor"
-    parent="imu_bottom_link"
-    namespace=""
-    x="${calibration['base_link']['imu_bottom_link']['sensor']['x']}"
-    y="${calibration['base_link']['imu_bottom_link']['sensor']['y']}"
-    z="${calibration['base_link']['imu_bottom_link']['sensor']['z']}"
-    roll="${calibration['base_link']['imu_bottom_link']['sensor']['roll']}"
-    pitch="${calibration['base_link']['imu_bottom_link']['sensor']['pitch']}"
-    yaw="${calibration['base_link']['imu_bottom_link']['sensor']['yaw']}"
-    fps="100"
   /> -->
 </robot>
