Commit message: update xacro

File: logiee-s-tc_sensor_kit_description/urdf/sensor_kit.xacro (robot description, xacro)
@@ -6,5 +6,5 @@
     <xacro:include filename="$(find camera_description)/urdf/monocular_camera.xacro"/>
     <xacro:include filename="$(find imu_description)/urdf/imu.xacro"/>
-    <xacro:arg name="gpu" default="false"/>
+    <xacro:arg name="gpu" default="true"/>
     <xacro:arg name="config_dir" default="$(find logiee-s-tc_sensor_kit_description)/config"/>
     <xacro:property name="sensor_kit_base_link" default="sensor_kit_base_link"/>
@@ -86,5 +86,5 @@
     <!-- imu -->
     <xacro:imu_macro
-      name="imu_link"
+      name="imu"
       parent="sensor_kit_base_link"
       namespace=""

File: logiee-s-tc_sensor_kit_description/urdf/sensors.xacro (robot description, xacro)
@@ -4,5 +4,5 @@
   <xacro:arg name="config_dir" default="$(find logiee-s-tc_sensor_kit_description)/config"/>
   <xacro:include filename="$(find logiee-s-tc_sensor_kit_description)/urdf/sensor_kit.xacro"/>
-  <xacro:property name="calibration" value="${load_yaml('$(arg config_dir)/sensors_calibration.yaml')}"/>
+  <xacro:property name="calibration" value="${xacro.load_yaml('$(arg config_dir)/sensors_calibration.yaml')}"/>
   <xacro:sensor_kit_macro parent="base_link" x="${calibration['base_link2sensor_kit_base_link']['x']}" y="${calibration['base_link2sensor_kit_base_link']['y']}" z="${calibration['base_link2sensor_kit_base_link']['z']}" roll="${calibration['base_link2sensor_kit_base_link']['roll']}" pitch="${calibration['base_link2sensor_kit_base_link']['pitch']}" yaw="${calibration['base_link2sensor_kit_base_link']['yaw']}" />
   <!-- <xacro:imu_macro
